File: dPicoTracker/dPicoTracker.kicad_pcb (KiCad board)
At the start: 2 copper layers, 23 parts, among them J1 Conn_01x02_Pin, P1 USB_C_Plug_USB2.0, U1 RP2040, U2 NCP1117-3.3_SOT223, U3 CJ431, U4 CJ431, U5 TPS61221DCK, U6 W25Q128JVS, X1 ABM8-272-T3

Commit message: make pcb
Parts:
- removed C1: 100nF, PCM_JLCPCB:C_1206
- removed C2, C6: 15pF, PCM_JLCPCB:C_1206
- removed C3, C4: 10µF, PCM_JLCPCB:C_1206
- removed J1: Conn_01x02_Pin, Connector_PinHeader_2.00mm:PinHeader_1x02_P2.00mm_Vertical
- removed P1: USB_C_Plug_USB2.0, Connector_USB:USB_C_Receptacle_XKB_U262-16XN-4BVC11
- removed R1, R2: 5.1kΩ, PCM_JLCPCB:R_1206
- removed R3, R4: 1kΩ, PCM_JLCPCB:R_1206
- removed U1: RP2040, Package_DFN_QFN:QFN-56-1EP_7x7mm_P0.4mm_EP3.2x3.2mm
- removed U2: NCP1117-3.3_SOT223, Package_TO_SOT_SMD:SOT-223-3_TabPin2
- removed U6: W25Q128JVS, Package_SO:SOIC-8_5.3x5.3mm_P1.27mm
- removed X1: ABM8-272-T3, footprints:ABM8-272-T3_ABR
- added A1: RaspberryPi_Pico, Module:RaspberryPi_Pico_Common_Unspecified, B.Cu at (60.1, 93.1)
- added AE1: HF 14MHz ANT, Connector_PinHeader_2.54mm:PinHeader_1x02_P2.54mm_Vertical, F.Cu at (63.7, 139.8)
- added AE2: VHF 144MHz ANT, Connector_PinHeader_2.54mm:PinHeader_1x02_P2.54mm_Vertical, F.Cu at (53.7, 139.5)
- added AE3: GPS_ANT, Connector_PinHeader_2.54mm:PinHeader_1x02_P2.54mm_Vertical, F.Cu at (47.8, 76.8)
- added C10: 100nF, Capacitor_SMD:C_1206_3216Metric, F.Cu at (55.0, 123.0)
- added C11: 240pF, Capacitor_SMD:C_1206_3216Metric, F.Cu at (66.2, 126.8)
- added C12: 430pF, Capacitor_SMD:C_1206_3216Metric, F.Cu at (66.2, 130.5)
- added C13: 240pF, Capacitor_SMD:C_1206_3216Metric, F.Cu at (67.0, 135.2)
- added C14: 24pF, Capacitor_SMD:C_1206_3216Metric, F.Cu at (54.5, 126.8)
- added C15: 43pF, Capacitor_SMD:C_1206_3216Metric, F.Cu at (54.5, 130.5)
- added C16: 24pF, Capacitor_SMD:C_1206_3216Metric, F.Cu at (53.7, 135.2)
- added C17: 100nF, Capacitor_SMD:C_1206_3216Metric, F.Cu at (72.5, 75.2)
- added C18: 100nF, Capacitor_SMD:C_1206_3216Metric, F.Cu at (72.2, 84.0)
- added C19: 100nF, Capacitor_SMD:C_1206_3216Metric, F.Cu at (63.8, 88.8)
- added C8: 100nF, Capacitor_SMD:C_1206_3216Metric, F.Cu at (55.5, 89.2)
- added C9: 100nF, Capacitor_SMD:C_1206_3216Metric, F.Cu at (64.5, 119.5)
- added IC1: ATGM336H-5N31, ATGM336H-5N31:ATGM336H5N31, F.Cu at (60.5, 80.2)
- added L2: 750nH, Inductor_SMD:L_1206_3216Metric, F.Cu at (62.5, 128.8)
- added L3: 750nH, Inductor_SMD:L_1206_3216Metric, F.Cu at (63.5, 134.3)
- added L4: 75nH, Inductor_SMD:L_1206_3216Metric, F.Cu at (58.2, 128.8)
- added L5: 75nH, Inductor_SMD:L_1206_3216Metric, F.Cu at (57.5, 134.3)
- added Q1: AO3401A, PCM_JLCPCB:Q_SOT-23, F.Cu at (61.2, 114.8)
- added Q2: AO3401A, PCM_JLCPCB:Q_SOT-23, F.Cu at (60.5, 88.4)
- added R11: 10kΩ, Resistor_SMD:R_1206_3216Metric, F.Cu at (55.0, 119.8)
- added R12: 10kΩ, Resistor_SMD:R_1206_3216Metric, F.Cu at (56.0, 117.0)
- added R14: 10kΩ, Resistor_SMD:R_1206_3216Metric, F.Cu at (72.0, 89.2)
- added R15: 10kΩ, Resistor_SMD:R_1206_3216Metric, F.Cu at (72.5, 70.2)
- added R7: 10kΩ, Capacitor_SMD:C_1206_3216Metric, F.Cu at (55.0, 97.2)
- added R8: 10kΩ, Resistor_SMD:R_1206_3216Metric, F.Cu at (61.5, 110.5)
- added R9: 10kΩ, Resistor_SMD:R_1206_3216Metric, F.Cu at (60.2, 91.8)
- added U7: MAX809STRG, footprints1:SOT-23_ONS, F.Cu at (54.5, 93.5)
- added U8: BMP280, Package_LGA:Bosch_LGA-8_2x2.5mm_P0.65mm_ClockwisePinNumbering, F.Cu at (72.5, 79.5)
- added Y1: Si5351A-B-GT, Package_SO:MSOP-10_3x3mm_P0.5mm, F.Cu at (60.0, 121.6)
- added Y2: XOS25026000LT00351005, Crystal:Crystal_SMD_2520-4Pin_2.5x2.0mm, F.Cu at (65.4, 116.0)
- C5, C7: footprint PCM_JLCPCB:C_1206 -> Capacitor_SMD:C_1206_3216Metric
- L1: footprint PCM_JLCPCB:L_1206 -> Inductor_SMD:L_1206_3216Metric
- R5: footprint PCM_JLCPCB:R_1206 -> Diode_SMD:D_1206_3216Metric
- R6: footprint PCM_JLCPCB:R_1206 -> Capacitor_SMD:C_1206_3216Metric
- U5: footprint Package_TO_SOT_SMD:SOT-23-5 -> Package_TO_SOT_SMD:Texas_R-PDSO-G6
- moved R6 160.0 mm to (47.0, 85.5), turned to 90 degrees
- moved R5 154.6 mm to (47.2, 95.8), turned to 90 degrees
- moved C7 154.1 mm to (47.2, 90.5), turned to 90 degrees
- moved U4 116.6 mm to (47.2, 105.2), turned to 180 degrees
- moved U3 116.5 mm to (47.2, 100.2)
- moved L1 56.8 mm to (61.7, 105.0)
- moved U5 50.1 mm to (62.0, 101.0)
- moved C5 37.5 mm to (58.0, 101.8), turned to 180 degrees
Connections:
- C5 pad 1: VBUS -> VCC
- L1 pad 1: VBUS -> VCC
- R5 pad 1: VBUS -> VCC
- U5 pad 1: VBUS -> VCC
Routing:
- net +3V3: track 0.00 -> 140.9 mm, vias 0 -> 1
- net /GPS_1PPS: track 0.00 -> 39.8 mm
- net /VFO_PWR_T: track 0.00 -> 35.9 mm, vias 0 -> 1
- net /VFO_3v3: track 0.00 -> 33.9 mm, vias 0 -> 2
- net /GPS_PWR_T: track 0.00 -> 31.3 mm
- net VCC: track 0.00 -> 30.3 mm, vias 0 -> 3
- net /VFO_SDA: track 0.00 -> 23.4 mm
- net GND: track 0.00 -> 21.2 mm, vias 0 -> 9
- net /VFO_SCL: track 0.00 -> 18.1 mm
- net Net-(IC1-VCC): track 0.00 -> 16.9 mm, vias 0 -> 2
- net /SENS_SDA: track 0.00 -> 15.5 mm
- net /UART1_RX: track 0.00 -> 15.5 mm
- net /VFO_CLK2: track 0.00 -> 14.8 mm
- net /UART1_TX: track 0.00 -> 14.1 mm
- net /GPS_RESET: track 0.00 -> 13.9 mm, vias 0 -> 1
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- added copper zone on B.Cu, net GND
- added copper zone on F.Cu, net GND
Other:
- board outline added: 32 x 76.1 mm

Commit message: Finish PCB i think
Parts:
- added J1: Conn_01x02_Pin, Connector_PinSocket_2.00mm:PinSocket_1x02_P2.00mm_Vertical, F.Cu at (46.1, 113.8)
- moved U3 0.82 mm to (48.1, 100.2)
- moved U4 0.76 mm to (48.0, 105.1)
Routing:
- net GND: track 21.2 -> 44.0 mm, vias 9 -> 11
- net VCC: track 30.3 -> 45.4 mm
- net /VFO_OSC: track 5.70 -> 6.39 mm
Other:
- board text added: "A"
- board text added: "GND"
- board text added: "VCC"
