File: direwolfTracker/direwolfTracker.kicad_pcb (KiCad board)
At the start: 2 copper layers, 32 x 53 mm, 25 parts, among them IC1 ATGM336H-5N31, J1 Raspberry_Pi_2_3, J11 Conn_01x04_Pin, J12 Conn_01x04_Pin, J3 Conn_01x02_Pin, J4 Conn_01x02_Pin, J7 Conn_01x04_Pin, J8 Conn_01x03_Pin, Q1 MMBT2222A, U1 TPS61222DCK, U2 ICM7555xP

Commit message: add version no
Other:
- board text added: "v1.0"
Changed lines of the file:
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@@
+		)
+	)
+	(gr_text "v1.0"
+		(at 60 62 0)
+		(layer "B.SilkS")
+		(effects
+			(font
+				(size 1 1)
+				(thickness 0.1)
+			)
+			(justify left bottom mirror)
 		)
 	)

Commit message: add BOMs
Other:
- board text added: "GPS"
- board text added: "Q1"
Changed lines of the file:
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@@
 		)
 		(property "Value" "MMBT2222A"
-			(at 0 2.4 90)
+			(at -1.01 2.87 90)
 			(layer "F.Fab")
 			(effects
@@
 		)
 		(fp_text user "${REFERENCE}"
-			(at 0 0 90)
-			(layer "F.Fab")
+			(at -0.2 0.01 90)
+			(layer "F.SilkS")
 			(effects
 				(font
@@
 		(tags "Through hole pin header THT 1x02 2.54mm single row")
 		(property "Reference" "AE3"
-			(at 0 -2.33 0)
+			(at -0.07 -4.005 0)
 			(layer "F.SilkS")
 			(effects
@@
 		(layer "Edge.Cuts")
 	)
+	(gr_text "GND"
+		(at 43.68 65.88 0)
+		(layer "F.SilkS")
+		(effects
+			(font
+				(size 1 1)
+				(thickness 0.1)
+			)
+			(justify left bottom)
+		)
+	)
 	(gr_text "G"
 		(at 47.45 53.1 0)
@@
 	)
 	(gr_text "SP"
+		(at 43.97 60.6 0)
+		(layer "F.SilkS")
+		(effects
+			(font
+				(size 1 1)
+				(thickness 0.1)
+			)
+			(justify left bottom)
+		)
+	)
+	(gr_text "SP"
 		(at 47.35 47.95 0)
 		(layer "F.SilkS")
@@
 		)
 	)
+	(gr_text "GPS"
+		(at 61.54 63.12 0)
+		(layer "F.SilkS")
+		(effects
+			(font
+				(size 1 1)
+				(thickness 0.1)
+			)
+			(justify left bottom)
+		)
+	)
+	(gr_text "MIC"
+		(at 43.84 63.41 0)
+		(layer "F.SilkS")
+		(effects
+			(font
+				(size 1 1)
+				(thickness 0.1)
+			)
+			(justify left bottom)
+		)
+	)
+	(gr_text "Q1"
+		(at 45.52 86.37 0)
+		(layer "F.SilkS")
+		(effects
+			(font
+				(size 1 1)
+				(thickness 0.1)
+			)
+			(justify left bottom)
+		)
+	)
 	(gr_text "5v"
 		(at 51.35 48.5 180)
@@
 		)
 	)
+	(gr_text "GND"
+		(at 61.46 70.61 0)
+		(layer "F.SilkS")
+		(effects
+			(font
+				(size 1 1)
+				(thickness 0.1)
+			)
+			(justify left bottom)
+		)
+	)
 	(gr_text "MIC"
 		(at 50.05 93.5 90)
@@
 		)
 	)
+	(gr_text "SP"
+		(at 39.6 60.9 270)
+		(layer "B.SilkS")
+		(effects
+			(font
+				(size 1 1)
+				(thickness 0.1)
+			)
+			(justify left bottom mirror)
+		)
+	)
+	(gr_text "GPS"
+		(at 64.64 63.09 0)
+		(layer "B.SilkS")
+		(effects
+			(font
+				(size 1 1)
+				(thickness 0.1)
+			)
+			(justify left bottom mirror)
+		)
+	)
 	(gr_text "Designed for Apex 2025\nMarcus Kauffman KN6UYL\nJoshua Truman\nHudson Hilal"
 		(at 60.1 74.75 0)
@@
 		)
 	)
+	(gr_text "GND"
+		(at 64.59 70.61 0)
+		(layer "B.SilkS")
+		(effects
+			(font
+				(size 1 1)
+				(thickness 0.1)
+			)
+			(justify left bottom mirror)
+		)
+	)
+	(gr_text "GND"
+		(at 55.5 49.63 0)
+		(layer "B.SilkS")
+		(effects
+			(font
+				(size 1 1)
+				(thickness 0.1)
+			)
+			(justify left bottom mirror)
+		)
+	)
+	(gr_text "GND"
+		(at 39.51 67.04 270)
+		(layer "B.SilkS")
+		(effects
+			(font
+				(size 1 1)
+				(thickness 0.1)
+			)
+			(justify left bottom mirror)
+		)
+	)
 	(gr_text "G"
 		(at 48.7 53.05 0)
@@
 		)
 	)
+	(gr_text "VBATT"
+		(at 61.17 50.56 0)
+		(layer "B.SilkS")
+		(effects
+			(font
+				(size 1 1)
+				(thickness 0.1)
+			)
+			(justify left bottom mirror)
+		)
+	)
+	(gr_text "5v"
+		(at 51.81 49.64 0)
+		(layer "B.SilkS")
+		(effects
+			(font
+				(size 1 1)
+				(thickness 0.1)
+			)
+			(justify left bottom mirror)
+		)
+	)
 	(gr_text "SPK"
 		(at 60.05 90.4 90)
@@
 	)
 	(gr_text "MIC"
+		(at 44.05 64.18 270)
+		(layer "B.SilkS")
+		(effects
+			(font
+				(size 1 1)
+				(thickness 0.1)
+			)
+			(justify left bottom mirror)
+		)
+	)
+	(gr_text "MIC"
 		(at 49.9 55.679 0)
 		(layer "B.SilkS")
 		(effects
+			(font
+				(size 1 1)
+				(thickness 0.1)
+			)
+			(justify left bottom mirror)
+		)
+	)
+	(gr_text "GND"
+		(at 61.41 47.63 0)
+		(layer "B.SilkS")
+		(effects
